Commit message: Increased size of box and cylinder

File: pcl_node/urdfs/box.urdf (robot description, URDF)
Before this commit: robot simple_box, 1 links, 0 joints
Links:
- link my_box: geometry collision box size=.2 0.2 0.2; visual box size=.2 0.2 0.2

File: pcl_node/urdfs/cylinder.urdf (robot description, URDF)
Before this commit: robot simple_box, 1 links, 0 joints
Links:
- link my_box: geometry collision cylinder length=0.2 radius=.1; visual cylinder length=0.2 radius=.1
