Commit message: Added sphere urdf and fixed naming issues in Cylinder urdf

File: pcl_node/urdfs/cylinder.urdf (robot description, URDF)
Before this commit: robot simple_box, 1 links, 0 joints
Links:
- removed link my_box
- added link my_cylinder, mass 1.0; collision cylinder length=0.2 radius=.1; visual cylinder length=0.2 radius=.1
