Commit message: cone works, pcl_node takes in param for switch case

File: pcl_node/urdfs/cone.urdf (robot description, URDF)
Before this commit: robot simple_cone, 1 links, 0 joints
Links:
- link my_cone: geometry collision mesh filename=package://pcl_node/urdfs/cone.STL scale=0.15 0.15 0.3; visual mesh filename=package://pcl_node/urdfs/cone.STL scale=0.15 0.15 0.3
